File: hardware/hawk.kicad_pcb (KiCad board)
At the start: 2 copper layers, 41 x 41 mm, 40 parts, among them J1 UART2, J2 SWD, J3 54-00298, SW1 EVQ-P7A01P, U1 AP7312-1833W6-7, U2 STM32G431K6Tx, U3 MAX9860ETG+T

Commit message: Initial Commit
Parts:
- added C20: 10uF, Capacitor_SMD:C_0603_1608Metric_Pad1.08x0.95mm_HandSolder, F.Cu at (132.1, 98.9)
- added H1: MountingHole, MountingHole:MountingHole_3.2mm_M3, F.Cu at (133.5, 114.5)
- added H2: MountingHole, MountingHole:MountingHole_3.2mm_M3, F.Cu at (164.5, 91.5)
- added U4: MIC5504-1.8YM5, Package_TO_SOT_SMD:SOT-23-5, F.Cu at (161.8, 110.0)
- R4: value 150 -> 1.5k
- SW1: value EVQ-P7A01P -> EVQ-P7L01P; footprint EVQ_P7A01P:EVQ_P7_PAN -> EVQ_P7L01P:EVQ_P7_PAN
- U1: value AP7312-1833W6-7 -> MIC5504-3.3YM5; footprint AP7312_1833W6_7:SOT26_DIO -> Package_TO_SOT_SMD:SOT-23-5
- moved R4 13.3 mm to (154.7, 97.8), turned to -90 degrees
- moved C1 8.12 mm to (153.7, 112.0), turned to 180 degrees
- moved G*** 5.11 mm to (156.8, 93.0)
- moved U1 2.87 mm to (161.8, 105.8), turned to 90 degrees
- moved C3 2.74 mm to (161.9, 102.9), turned to 0 degrees
- moved C9 2.56 mm to (138.6, 98.9)
- moved J2 2.53 mm to (166.0, 107.7)
- moved TP4 2.25 mm to (148.9, 117.9)
- moved TP3 2.25 mm to (151.1, 117.9)
- moved J1 1.98 mm to (162.3, 100.6)
- moved NT1 1.98 mm to (141.2, 113.2)
- moved C4 1.81 mm to (157.5, 98.6)
- moved R3 1.79 mm to (157.5, 97.0), turned to 180 degrees
- moved C6 1.74 mm to (158.4, 110.8), turned to -90 degrees
- moved C2 1.28 mm to (161.8, 113.0), turned to 180 degrees
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Connections:
- C9 pad 1: Net-(C9-Pad1) -> /MIC
- J2 pad 4: /SDOUT -> /SWDIO
- J3 pad 1: Net-(C9-Pad1) -> /MIC
- J3 pad 3: Net-(U3-OUTP) -> /SPKR
- J3 pad 4: Net-(U3-OUTP) -> /SPKR
- R3 pad 2: +5V -> +3V3
- R4 pad 1: /SDOUT -> Net-(U2-PB0)
- R4 pad 2: Net-(U3-SDOUT) -> GND
- R5 pad 1: Net-(U3-MICLP) -> /MIC
- SW1 pad 1: Net-(U2-PB0) -> +3V3
- SW1 pad 1*: Net-(U2-PB0) -> unconnected-(SW1-Pad1*)
- SW1 pad 2: GND -> unconnected-(SW1-Pad2)
- SW1 pad 2*: GND -> Net-(U2-PB0)
- U1 pad 1: +3V3 -> +5V
- U1 pad 4: +5V -> unconnected-(U1-NC-Pad4)
- U1 pad 5: +5V -> +3V3
- U2 pad 18: /BCLK -> /MCLK
- U2 pad 19: /LPCLK -> unconnected-(U2-PA9-Pad19)
- U2 pad 23: /SDOUT -> /SWDIO
- U2 pad 25: unconnected-(U2-PA15-Pad25) -> /I2C1_SCL
- U2 pad 26: unconnected-(U2-PB3-Pad26) -> /BCLK
- U2 pad 28: unconnected-(U2-PB5-Pad28) -> /SDOUT
- U2 pad 31: /I2C1_SCL -> Net-(U2-PB0)
- U2 pad 8: /MCLK -> unconnected-(U2-PA3-Pad8)
- U2 pad 9: unconnected-(U2-PA4-Pad9) -> /LPCLK
- U3 pad 15: Net-(U3-SDOUT) -> /SDOUT
- U3 pad 20: GNDA -> unconnected-(U3-MICRN-Pad20)
- U3 pad 21: GNDA -> unconnected-(U3-MICRP-Pad21)
- U3 pad 8: GNDA -> unconnected-(U3-OUTN-Pad8)
Routing:
- net GND: track 46.5 -> 16.6 mm
- net /SPKR: track 0.00 -> 25.1 mm, vias 0 -> 1
- net /SWDIO: track 0.00 -> 24.1 mm, vias 0 -> 1
- net +3V3: track 60.3 -> 84.0 mm, vias 2 -> 5
- net /MIC: track 0.00 -> 21.5 mm
- net Net-(C9-Pad1): track 18.2 -> 0.00 mm
- net Net-(U3-OUTP): track 30.0 -> 15.2 mm
- net /I2C1_SCL: track 26.8 -> 16.8 mm, vias 2 -> 0
- net /BCLK: track 9.39 -> 18.9 mm, vias 0 -> 2
- net /LPCLK: track 9.56 -> 18.5 mm, vias 0 -> 2
- net /SDOUT: track 24.9 -> 16.9 mm, vias 3 -> 2
- net GNDA: track 21.6 -> 13.8 mm
- net /MCLK: track 19.5 -> 11.8 mm
- net Net-(U2-PB0): track 30.5 -> 38.1 mm, vias 1 -> 4
- net +5V: track 32.9 -> 25.3 mm, vias 2 -> 0
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Other:
- outline, holes or cut-outs redrawn
- board text added: "Hawk By Ryzee119"
- board text removed: "By Ryzee119 Hawk"
