File: hardware/hawk.kicad_sch (KiCad schematic)
At the start: 37 parts, among them J1 UART2, J2 SWD, J3 54-00298, SW1 EVQ-P7A01P, U1 AP7312-1833W6-7, U2 STM32G431K6Tx, U3 MAX9860ETG+T

Commit message: Initial Commit
Parts:
- removed U1: AP7312-1833W6-7, SOT26_DIO, symbol AP7312_1833W6_7:AP7312-1833W6-7
- added C20: 10uF, Capacitor_SMD:C_0603_1608Metric_Pad1.08x0.95mm_HandSolder, symbol Device:C
- added H1, H2: MountingHole, MountingHole:MountingHole_3.2mm_M3, symbol Mechanical:MountingHole
- added U1: MIC5504-3.3YM5, Package_TO_SOT_SMD:SOT-23-5, symbol Regulator_Linear:MIC5504-3.3YM5
- added U4: MIC5504-1.8YM5, Package_TO_SOT_SMD:SOT-23-5, symbol Regulator_Linear:MIC5504-1.8YM5
- R4: value 150 -> 1.5k
- SW1: value EVQ-P7A01P -> EVQ-P7L01P; footprint EVQ_P7_PAN -> EVQ_P7L01P:EVQ_P7_PAN; symbol EVQ_P7A01P:EVQ-P7A01P -> EVQ_P7L01P:EVQ-P7L01P
- U3: footprint 21-0139I_T2444-4_MXM -> MAX9860:21-0139I_T2444-4_MXM
Connections:
- net +1V8: now also U4.5 (VOUT)
- net +3V3: now also R3.2, SW1.1, U1.5 (VOUT)
- net +5V: now also U1.1 (VIN), U1.3 (EN), U4.1 (VIN), U4.3 (EN); no longer R3.2
- net BCLK: now also U2.26 (PB3); no longer U2.18 (PA8)
- net GND: now also R4.2, U1.2 (GND), U4.2 (GND); no longer SW1.2, SW1.2*
- net GNDA: no longer U3.20 (MICRN), U3.21 (MICRP), U3.8 (OUTN)
- net I2C1_SCL: now also U2.25 (PA15); no longer U2.31 (PB8)
- net LPCLK: now also U2.9 (PA4); no longer U2.19 (PA9)
- net MCLK: now also U2.18 (PA8); no longer U2.8 (PA3)
- net SDOUT: now also U2.28 (PB5), U3.15 (SDOUT); no longer J2.4 (Pin_4), R4.1, U2.23 (PA13)
- net MIC: now reaches C9.1, J3.1
- net MIC: now also R5.1
- net at C9.2, U3.23 (MICLP): no longer R5.1
- net SPKR: now reaches J3.3, J3.4
- net SPKR: now also C20.1; no longer U3.7 (OUTP)
- new net: R4.1, SW1.2*, U2.13 (PB0), U2.31 (PB8)
- new net: C20.2, U3.7 (OUTP)
- new net SWDIO: J2.4 (Pin_4), U2.23 (PA13)
- now unconnected: SW1.1*
Other:
- company: Ryan Wendland -> Ryzee119
- moved on the sheet: C1, C2, J2, SW1
